File: Cr0wn60.kicad_pcb (KiCad board)
At the start: 2 copper layers, 285.8 x 95.2 mm, 174 parts, among them J1 Conn_01x04_MountingPin, J2 Conn_01x02, SW1 SW_Push_45deg, SW10 SW_Push_45deg, SW12 SW_Push_45deg, SW13 SW_Push_45deg, SW14 SW_Push_45deg, SW15 SW_Push_45deg, SW16 SW_Push_45deg, SW17 SW_Push_45deg, SW2 SW_Push_45deg, SW20 SW_Push_45deg, SW21 SW_Push_45deg, SW23 SW_Push_45deg, SW24 SW_Push_45deg, SW25 SW_Push_45deg, SW26 SW_Push_45deg, SW3 SW_Push_45deg, SW30 SW_Push_45deg, SW31 SW_Push_45deg, SW32 SW_Push_45deg, SW34 SW_Push_45deg, SW35 SW_Push_45deg, SW36 SW_Push_45deg, SW37 SW_Push_45deg, SW4 SW_Push_45deg, SW40 SW_Push_45deg, SW41 SW_Push_45deg, SW42 SW_Push_45deg, SW43 SW_Push_45deg, SW45 SW_Push_45deg, SW46 SW_Push_45deg, SW5 SW_Push_45deg, SW50 SW_Push_45deg, SW51 SW_Push_45deg, SW52 SW_Push_45deg, SW53 SW_Push_45deg, SW54 SW_Push_45deg, SW56 SW_Push_45deg, SW57 SW_Push_45deg, SW6 SW_Push_45deg, SW60 SW_Push_45deg, SW61 SW_Push_45deg, SW62 SW_Push_45deg, SW63 SW_Push_45deg, SW64 SW_Push_45deg, SW65 SW_Push_45deg, SW70 SW_Push_45deg, SW71 SW_Push_45deg, SW72 SW_Push_45deg, SW73 SW_Push_45deg, SW74 SW_Push_45deg, SW75 SW_Push_45deg, SW76 SW_Push_45deg, SW80 SW_Push_45deg, SW81 SW_Push_45deg, SW82 SW_Push_45deg, SW83 SW_Push_45deg, SW84 SW_Push_45deg, SW85 SW_Push_45deg, SW86 SW_Push_45deg, SW87 SW_Push_45deg, U1 AMS1117, U2 W25Q128JVS, U3 RP2040_QFN_56, Y1 Crystal_Small

Commit message: add production files
Parts:
- C11: value C_Small -> 0.1u
- C12, C13: value C_Small -> 27p
- LED1, LED10, LED11, LED12, LED13, LED14, LED15, LED2, LED3, LED4, LED5, LED6, LED7, LED8, LED9: moved to B.Cu
- R1, R2: value R_Small -> 22
- R3, R4, R5: value R_Small -> 1k
- Y1: value Crystal_Small -> 12M
- turned LED1 to 180 degrees
- turned LED10 to 90 degrees
- turned LED11 to 90 degrees
- turned LED12 to 180 degrees
- turned LED13 to 180 degrees
- turned LED14 to 180 degrees
- turned LED15 to 180 degrees
- turned LED2 to 180 degrees
- turned LED3 to 180 degrees
- turned LED4 to -90 degrees
- turned LED5 to -90 degrees
- turned LED6 to 0 degrees
- turned LED7 to 0 degrees
- turned LED8 to 0 degrees
- turned LED9 to 0 degrees
Routing:
- net Net-(LED5-I): track 101.3 -> 95.8 mm
- net /LED: track 35.0 -> 39.9 mm
- net Net-(LED6-I): track 59.0 -> 62.5 mm
- net Net-(LED11-I): track 35.0 -> 31.6 mm
- net Net-(LED10-O): track 50.0 -> 47.2 mm
- net Net-(LED7-I): track 59.0 -> 61.6 mm
- net Net-(LED3-I): track 35.3 -> 32.9 mm
- net Net-(LED12-I): track 26.0 -> 27.8 mm
- net Net-(LED8-I): track 68.2 -> 66.7 mm
- net /P3: track 497.5 -> 496.1 mm
- net Net-(LED2-I): track 36.8 -> 37.8 mm
- net Net-(LED14-I): track 52.5 -> 51.9 mm, vias 2 -> 0
- net +5V: track 44.1 -> 43.6 mm
- net (no net): vias 1 -> 0
