File: Cr0wn60.kicad_pcb (KiCad board)
At the start: 2 copper layers, 285.8 x 95.2 mm, 174 parts, among them J1 Conn_01x04_MountingPin, J2 Conn_01x02, SW1 SW_Push_45deg, SW10 SW_Push_45deg, SW12 SW_Push_45deg, SW13 SW_Push_45deg, SW14 SW_Push_45deg, SW15 SW_Push_45deg, SW16 SW_Push_45deg, SW17 SW_Push_45deg, SW2 SW_Push_45deg, SW20 SW_Push_45deg, SW21 SW_Push_45deg, SW23 SW_Push_45deg, SW24 SW_Push_45deg, SW25 SW_Push_45deg, SW26 SW_Push_45deg, SW3 SW_Push_45deg, SW30 SW_Push_45deg, SW31 SW_Push_45deg, SW32 SW_Push_45deg, SW34 SW_Push_45deg, SW35 SW_Push_45deg, SW36 SW_Push_45deg, SW37 SW_Push_45deg, SW4 SW_Push_45deg, SW40 SW_Push_45deg, SW41 SW_Push_45deg, SW42 SW_Push_45deg, SW43 SW_Push_45deg, SW45 SW_Push_45deg, SW46 SW_Push_45deg, SW5 SW_Push_45deg, SW50 SW_Push_45deg, SW51 SW_Push_45deg, SW52 SW_Push_45deg, SW53 SW_Push_45deg, SW54 SW_Push_45deg, SW56 SW_Push_45deg, SW57 SW_Push_45deg, SW6 SW_Push_45deg, SW60 SW_Push_45deg, SW61 SW_Push_45deg, SW62 SW_Push_45deg, SW63 SW_Push_45deg, SW64 SW_Push_45deg, SW65 SW_Push_45deg, SW70 SW_Push_45deg, SW71 SW_Push_45deg, SW72 SW_Push_45deg, SW73 SW_Push_45deg, SW74 SW_Push_45deg, SW75 SW_Push_45deg, SW76 SW_Push_45deg, SW80 SW_Push_45deg, SW81 SW_Push_45deg, SW82 SW_Push_45deg, SW83 SW_Push_45deg, SW84 SW_Push_45deg, SW85 SW_Push_45deg, SW86 SW_Push_45deg, SW87 SW_Push_45deg, U1 AMS1117, U2 W25Q128JVS, U3 RP2040_QFN_56, Y1 12M

Commit message: update
Parts:
- SWR0, SWR1: moved to F.Cu
- moved SWR1 14.8 mm to (133.2, 9.40), turned to 180 degrees
- moved SWR0 12.8 mm to (99.0, 9.53), turned to 0 degrees
- moved R4 8.09 mm to (129.0, 10.2), turned to 180 degrees
Routing:
- net +3V3: track 27.4 -> 17.1 mm, vias 4 -> 2
- net /MCU/RUN: track 27.6 -> 23.3 mm, vias 2 -> 1
- net /LED: track 39.9 -> 36.1 mm
- net /P0: track 345.8 -> 348.8 mm
- net /P1: track 407.6 -> 409.7 mm
- net GND: track 22.0 -> 20.0 mm, vias 39 -> 37
- net /MCU/QSPI_SS: track 20.9 -> 22.8 mm
- net /MCU/BOOTSEL: track 2.91 -> 1.77 mm, vias 0 -> 1

Commit message: some tweak
Parts:
- removed the REF** at (97.6, 76.2)
- added REF**: KBD_CASE, ADeL_kbd:KBD_CASE, F.Cu at (128.6, 38.1)
- SW83: footprint SMKJP:SW_Cherry_MX1A_2.25u_PCB -> SMKJP:SW_Cherry_MX1A_1.75u_PCB
- SW86, SW87: footprint SMKJP:SW_Cherry_MX1A_1.25u_PCB -> SMKJP:SW_Cherry_MX1A_1.50u_PCB
- moved DK85 9.53 mm to (156.8, 81.3)
- moved REF** 9.53 mm to (131.0, 76.2)
- moved SW84 9.53 mm to (131.0, 76.2)
- moved DK84 9.52 mm to (125.9, 81.3)
- moved SW85 9.52 mm to (161.9, 76.2)
- moved LED7 7.24 mm to (111.8, 83.3)
- moved DK86 7.14 mm to (180.7, 81.3)
- moved LED8 7.14 mm to (175.0, 83.3)
- moved SW86 7.14 mm to (185.7, 76.2)
- moved DK83 4.76 mm to (87.8, 81.3)
- moved SW83 4.76 mm to (92.9, 76.2)
- moved DR8 4.25 mm to (126.7, 69.8)
- moved DK87 2.38 mm to (209.2, 81.3)
- moved SW87 2.38 mm to (214.3, 76.2)
Routing:
- net /P5: track 390.2 -> 402.9 mm
- net Net-(LED6-I): track 62.5 -> 52.8 mm
- net Net-(LED8-I): track 66.7 -> 73.9 mm
- net /P6: track 346.9 -> 353.9 mm
- net /P8: track 62.5 -> 67.4 mm
- net Net-(DR8-K): track 197.9 -> 193.9 mm
- net /P4: track 380.3 -> 377.5 mm
- net /P7: track 261.2 -> 258.7 mm
- net /P3: track 496.1 -> 495.5 mm, vias 14 -> 15
- net Net-(LED7-I): track 61.6 -> 61.0 mm
