File: KEYMATRIX.kicad_sch (KiCad schematic)
At the start: 129 parts, among them SW1 SW_Push_45deg, SW10 SW_Push_45deg, SW12 SW_Push_45deg, SW13 SW_Push_45deg, SW14 SW_Push_45deg, SW15 SW_Push_45deg, SW16 SW_Push_45deg, SW17 SW_Push_45deg, SW2 SW_Push_45deg, SW20 SW_Push_45deg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

Commit message: update
Parts:
- removed DR0: D_Small, Diode_SMD:D_SOD-123, symbol Device:D_Small
- added D2: D_Small, symbol Device:D_Small
Connections:
- net P0: now also D2.2 (A)
- net at SW1.2, SW2.2, SW3.2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: now also D2.1 (K)
