File: MCU.kicad_sch (KiCad schematic)
At the start: 27 parts, among them J1 Conn_01x04_MountingPin, J2 Conn_01x02, U1 AMS1117, U2 W25Q128JVS, U3 RP2040_QFN_56, Y1 Crystal_Small

Commit message: update
Parts:
- added R6: R_Small, symbol Device:R_Small
Connections:
- net +3V3: now also R6.1
- net RUN: now also R6.2
Other:
- moved on the sheet: R4, SWR0, SWR1, U2
